File: Kicad Files/Kicad Files.kicad_pcb (KiCad board)
At the start: 2 copper layers, 300.1 x 90.5 mm, 71 parts, among them J1 USB_C_Receptacle_USB2.0_16P, J2 Conn_01x04_Socket, J3 PCM5102, J4 PAM8302, J5 DAC_OUT, SW1 SW_Push, SW10 SW_Push, SW11 SW_Push, SW12 SW_Push, SW13 SW_Push, SW14 SW_Push, SW15 SW_Push, SW16 SW_Push, SW17 SW_Push, SW18 SW_Push, SW19 SW_Push, SW2 SW_Push, SW20 SW_Push, SW21 SW_Push, SW22 SW_Push, SW23 SW_Push, SW24 SW_Push, SW25 SW_Push, SW3 SW_Push, SW4 SW_Push, SW5 SW_Push, SW6 SW_Push, SW7 SW_Push, SW8 SW_Push, SW9 SW_Push, U1 4051

Commit message: wire more of the pcb
Parts:
- moved RV8 96.5 mm to (201.5, 111.5), turned to -90 degrees
- moved J2 87.4 mm to (220.4, 112.0)
- moved RV7 81.5 mm to (187.0, 111.5), turned to -90 degrees
- moved RV6 66.0 mm to (172.5, 111.5), turned to -90 degrees
- moved RV5 50.5 mm to (158.0, 111.5), turned to -90 degrees
- moved J4 35.5 mm to (298.0, 125.1), turned to 180 degrees
- moved RV4 35.0 mm to (143.5, 111.5), turned to -90 degrees
- moved J5 33.2 mm to (303.5, 116.3), turned to 0 degrees
- moved RV3 19.5 mm to (129.0, 111.5), turned to -90 degrees
- moved RV1 11.5 mm to (100.0, 111.5), turned to -90 degrees
- moved D12 7.50 mm to (144.0, 171.0), turned to 180 degrees
- moved J3 7.32 mm to (304.1, 143.0)
- moved RV2 4.00 mm to (114.5, 111.5), turned to -90 degrees
- moved A1 3.11 mm to (60.5, 122.1)
Routing:
- net /COL4: track 0.00 -> 431.4 mm, vias 0 -> 4
- net /COL2: track 0.00 -> 387.3 mm, vias 0 -> 4
- net /COL1: track 0.00 -> 349.8 mm, vias 0 -> 4
- net /COL3: track 0.00 -> 335.9 mm, vias 0 -> 4
- net /COL0: track 0.00 -> 330.2 mm
- net /ROW4: track 0.00 -> 310.7 mm, vias 0 -> 1
- net /ROW3: track 0.00 -> 254.8 mm, vias 0 -> 1
- net +3V3: track 0.00 -> 229.1 mm, vias 0 -> 2
- net /ROW2: track 0.00 -> 203.8 mm, vias 0 -> 1
- net /ROW1: track 0.00 -> 159.7 mm, vias 0 -> 1
- net /OLED_SCL: track 0.00 -> 153.1 mm, vias 0 -> 2
- net /OLED_SDA: track 0.00 -> 151.7 mm
- net /ROW0: track 0.00 -> 133.3 mm, vias 0 -> 1
- net Net-(J1-CC1): track 0.00 -> 55.6 mm, vias 0 -> 1
- net Net-(F1-Pad2): track 0.00 -> 49.9 mm
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
Commit message: add decor and finish wire
Parts:
- added ?: LOGO, images:crotchet, F.Cu at (279.1, 141.6)
- added ?: LOGO, images:halflifeimage, F.Cu at (255.0, 116.0)
- added ?: LOGO, images:quaver, F.Cu at (294.7, 151.3)
- added ?: LOGO, images:quaver + semiquaver, F.Cu at (286.0, 142.0)
- added ?: LOGO, images:profilepicture, F.Cu at (314.0, 171.5)
Routing:
- net +5V: track 34.9 -> 334.2 mm, vias 2 -> 3
- net /I2S_DIN: track 0.00 -> 275.7 mm, vias 0 -> 3
- net /I2S_BCK: track 0.00 -> 266.5 mm, vias 0 -> 3
- net /I2S_LRCK: track 0.00 -> 265.3 mm, vias 0 -> 4
- net /MUX_A: track 0.00 -> 181.2 mm, vias 0 -> 2
- net /MUX_B: track 0.00 -> 170.4 mm, vias 0 -> 2
- net /KNOBS: track 0.00 -> 159.4 mm
- net /MUX_C: track 0.00 -> 156.6 mm, vias 0 -> 2
- net /POT0: track 0.00 -> 121.9 mm
- net /POT1: track 0.00 -> 109.2 mm, vias 0 -> 1
- net /POT2: track 0.00 -> 92.6 mm, vias 0 -> 1
- net /POT3: track 0.00 -> 83.8 mm, vias 0 -> 2
- net GND: track 0.00 -> 71.2 mm, vias 0 -> 7
- net /POT5: track 0.00 -> 64.5 mm, vias 0 -> 3
- net /POT4: track 0.00 -> 58.5 mm, vias 0 -> 2
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- added copper zone on B.Cu, net GND
- added copper zone on F.Cu, net GND
Other:
- board text added: "●●●"

Commit message: readme pushing
Other:
- board text added: "ATTACK"
- board text added: "ECHO"
- board text added: "INSTR"
- board text added: "OCTAVE"
- board text added: "RELEASE"
- board text added: "TONE"
- board text added: "TRANSPOSE"
- board text added: "VOLUME"
Changed lines of the file:
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@@
 			(outputformat 1)
 			(mirror no)
-			(drillshape 1)
+			(drillshape 0)
 			(scaleselection 1)
-			(outputdirectory "")
+			(outputdirectory "../Gerbers/")
 		)
 	)
@@
 		(layer "Edge.Cuts")
 	)
+	(gr_text "RELEASE\n"
+		(at 150.5 127 0)
+		(layer "F.SilkS")
+		(effects
+			(font
+				(size 1.5 1.5)
+				(thickness 0.375)
+			)
+			(justify left bottom)
+		)
+	)
+	(gr_text "VOLUME\n"
+		(at 91.5 128 0)
+		(layer "F.SilkS")
+		(effects
+			(font
+				(size 2 2)
+				(thickness 0.4)
+			)
+			(justify left bottom)
+		)
+	)
+	(gr_text "INSTR \n"
+		(at 107.5 128 0)
+		(layer "F.SilkS")
+		(effects
+			(font
+				(size 2 2)
+				(thickness 0.4)
+			)
+			(justify left bottom)
+		)
+	)
+	(gr_text "TONE\n"
+		(at 122 128 0)
+		(layer "F.SilkS")
+		(effects
+			(font
+				(size 2 2)
+				(thickness 0.4)
+			)
+			(justify left bottom)
+		)
+	)
+	(gr_text "ATTACK\n"
+		(at 135.5 128 0)
+		(layer "F.SilkS")
+		(effects
+			(font
+				(size 2 2)
+				(thickness 0.4)
+			)
+			(justify left bottom)
+		)
+	)
+	(gr_text "ECHO\n"
+		(at 164.5 127.5 0)
+		(layer "F.SilkS")
+		(effects
+			(font
+				(size 2 2)
+				(thickness 0.4)
+			)
+			(justify left bottom)
+		)
+	)
+	(gr_text "OCTAVE\n"
+		(at 179 128 0)
+		(layer "F.SilkS")
+		(effects
+			(font
+				(size 2 2)
+				(thickness 0.4)
+			)
+			(justify left bottom)
+		)
+	)
+	(gr_text "TRANSPOSE\n"
+		(at 210 125 90)
+		(layer "F.SilkS")
+		(effects
+			(font
+				(size 2 2)
+				(thickness 0.4)
+			)
+			(justify left bottom)
+		)
+	)
 	(gr_text "●●●"
 		(at 299.5 153.5 -27)
@@
 		)
 		(min_thickness 0.25)
-		(fill
+		(fill yes
 			(thermal_gap 0.5)
 			(thermal_bridge_width 0.5)

Commit message: newbom for grant/self funded stuff
Connections:
- J4 pad 1: +5V -> GND
- J4 pad 2: GND -> +5V
Routing:
- net +5V: track 334.2 -> 327.4 mm
Changed lines of the file:
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@@
 			(layers "*.Cu" "*.Mask")
 			(remove_unused_layers no)
-			(net "+5V")
+			(net "GND")
 			(pinfunction "Pin_1_1")
 			(pintype "passive")
@@
 			(layers "*.Cu" "*.Mask")
 			(remove_unused_layers no)
-			(net "GND")
+			(net "+5V")
 			(pinfunction "Pin_2_2")
 			(pintype "passive")
@@
 	)
 	(segment
-		(start 40.34 108.5)
-		(end 80.5 108.5)
+		(start 24 129.5)
+		(end 26.5 129.5)
 		(width 0.25)
 		(layer "F.Cu")
@@
 	)
 	(segment
-		(start 298 125.12)
-		(end 304.15 131.27)
+		(start 40.34 108.5)
+		(end 81 108.5)
 		(width 0.25)
 		(layer "F.Cu")
@@
 	)
 	(segment
-		(start 24 129.5)
-		(end 26.5 129.5)
+		(start 298 122.58)
+		(end 304.15 128.73)
 		(width 0.25)
 		(layer "F.Cu")
@@
 	)
 	(segment
-		(start 304.15 131.27)
-		(end 304.15 143)
+		(start 36.42 112.42)
+		(end 36.34 112.5)
 		(width 0.25)
 		(layer "F.Cu")
@@
 	(segment
 		(start 36.42 112.42)
-		(end 36.34 112.5)
+		(end 40.34 108.5)
 		(width 0.25)
 		(layer "F.Cu")
@@
 	)
 	(segment
-		(start 36.42 112.42)
-		(end 40.34 108.5)
+		(start 24 129.5)
+		(end 27 132.5)
 		(width 0.25)
 		(layer "F.Cu")
@@
 	)
 	(segment
-		(start 24 129.5)
-		(end 27 132.5)
+		(start 304.15 143)
+		(end 304.5 142.65)
+		(width 0.25)
+		(layer "F.Cu")
+		(net "+5V")
+	)
+	(segment
+		(start 304.15 128.73)
+		(end 304.15 143)
 		(width 0.25)
 		(layer "F.Cu")
@@
 	)
 	(via
-		(at 80.5 108.5)
+		(at 81 108.5)
 		(size 0.6)
 		(drill 0.3)
@@
 	)
 	(segment
-		(start 26.5 129.5)
-		(end 29.5 129.5)
-		(width 0.25)
-		(layer "B.Cu")
-		(net "+5V")
-	)
-	(segment
-		(start 291.5 124.5)
-		(end 292.12 125.12)
-		(width 0.25)
-		(layer "B.Cu")
-		(net "+5V")
-	)
-	(segment
 		(start 83 108.5)
 		(end 83.5 109)
@@
 	)
 	(segment
-		(start 291 109)
-		(end 291.5 109.5)
-		(width 0.25)
-		(layer "B.Cu")
-		(net "+5V")
-	)
-	(segment
-		(start 291.5 109.5)
-		(end 291.5 124.5)
+		(start 26.5 129.5)
+		(end 29.5 129.5)
 		(width 0.25)
 		(layer "B.Cu")
@@
 	)
 	(segment
-		(start 83.5 109)
-		(end 291 109)
+		(start 81 108.5)
+		(end 83 108.5)
 		(width 0.25)
 		(layer "B.Cu")
@@
 	)
 	(segment
-		(start 292.12 125.12)
-		(end 298 125.12)
+		(start 284.42 109)
+		(end 298 122.58)
 		(width 0.25)
 		(layer "B.Cu")
@@
 	)
 	(segment
-		(start 80.5 108.5)
-		(end 83 108.5)
+		(start 83.5 109)
+		(end 284.42 109)
 		(width 0.25)
 		(layer "B.Cu")
