File: Kicad Files/Kicad Files.kicad_sch (KiCad schematic)
At the start: 68 parts, among them J1 USB_C_Receptacle_USB2.0_16P, J2 Conn_01x04_Socket, SW1 SW_Push, SW10 SW_Push, SW11 SW_Push, SW12 SW_Push, SW13 SW_Push, SW14 SW_Push, SW15 SW_Push, SW16 SW_Push, SW17 SW_Push, SW18 SW_Push, SW19 SW_Push, SW2 SW_Push, SW20 SW_Push, SW21 SW_Push, SW22 SW_Push, SW23 SW_Push, SW24 SW_Push, SW25 SW_Push, SW3 SW_Push, SW4 SW_Push, SW5 SW_Push, SW6 SW_Push, SW7 SW_Push, SW8 SW_Push, SW9 SW_Push, U1 4051

Commit message: finish schematics + footprints. arranged pcb in editor, but not wired
Parts:
- added J3: PCM5102, Connector_PinSocket_2.54mm:PinSocket_1x06_P2.54mm_Vertical, symbol Connector:Conn_01x06_Socket
- added J4: PAM8302, Connector_PinSocket_2.54mm:PinSocket_1x05_P2.54mm_Vertical, symbol Connector:Conn_01x05_Socket
- added J5: DAC_OUT, Connector_PinSocket_2.54mm:PinSocket_1x03_P2.54mm_Vertical, symbol Connector:Conn_01x03_Socket
- D1: footprint Package_SON:WSON-6-1EP_2x2mm_P0.65mm_EP1x1.6mm -> Diode_SMD:D_SMA_Handsoldering
- D10, D11, D12, D13, D14, D15, D16, D17, D18, D19, D2, D20, D21, D22, D23, D24, D25, D26, D3, D4, D5, D6, D7, D8, D9: footprint (none) -> Diode_THT:D_DO-35_SOD27_P7.62mm_Horizontal
- F1: footprint Package_SO:TSSOP-20_4.4x6.5mm_P0.65mm -> Fuse:Fuse_1206_3216Metric_Pad1.42x1.75mm_HandSolder
- J1: footprint Package_DFN_QFN:WDFN-10-1EP_3x3mm_P0.5mm_EP1.8x2.5mm -> Connector_USB:USB_C_Receptacle_HRO_TYPE-C-31-M-12
- J2: footprint (none) -> Connector_PinSocket_2.54mm:PinSocket_1x04_P2.54mm_Vertical
- R1, R2, R3, R4: footprint (none) -> Resistor_THT:R_Axial_DIN0207_L6.3mm_D2.5mm_P7.62mm_Horizontal
- RV1, RV2, RV3, RV4, RV5, RV6, RV7, RV8: footprint Resistor_THT:R_Array_SIP4 -> Potentiometer_THT:Potentiometer_Alps_RK09K_Single_Vertical
- SW1, SW10, SW11, SW12, SW13, SW14, SW15, SW16, SW17, SW18, SW19, SW2, SW20, SW21, SW22, SW23, SW24, SW25, SW3, SW4, SW5, SW6, SW7, SW8, SW9: footprint Button_Switch_SMD:Nidec_Copal_CAS-120A -> Button_Switch_Keyboard:SW_Cherry_MX_1.00u_PCB
- U1: footprint (none) -> Package_DIP:DIP-16_W7.62mm
Connections:
- net +5V: now also J3.1 (Pin_1), J4.1 (Pin_1)
- net GND: now also J3.2 (Pin_2), J3.6 (Pin_6), J4.2 (Pin_2), J4.4 (Pin_4), J5.2 (Pin_2); no longer A1.TP1 (USB_GND)
- net I2S_BCK: now reaches A1.24 (GPIO18)
- net I2S_BCK: now also J3.5 (Pin_5)
- net I2S_LRCK: now reaches A1.25 (GPIO19)
- net I2S_LRCK: now also J3.3 (Pin_3)
- net I2S_DIN: now reaches A1.26 (GPIO20)
- net I2S_DIN: now also J3.4 (Pin_4)
- new net AUDIO_L: J4.5 (Pin_5), J5.1 (Pin_1)
- no-connect marks 2 -> 21
Other:
- note added: "Amplifier"
- note added: "Digital to Analog Converter"

Commit message: newbom for grant/self funded stuff
Connections:
- net +5V: now also J4.2 (Pin_2); no longer J4.1 (Pin_1)
- net GND: now also J4.1 (Pin_1); no longer J4.2 (Pin_2)
Changed lines of the file:
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@@
 	)
 	(symbol
+		(lib_id "power:+5V")
+		(at 129.54 85.09 90)
+		(unit 1)
+		(body_style 1)
+		(exclude_from_sim no)
+		(in_bom yes)
+		(on_board yes)
+		(in_pos_files yes)
+		(dnp no)
+		(fields_autoplaced yes)
+		(property "Reference" "#PWR035"
+			(at 133.35 85.09 0)
+			(hide yes)
+			(show_name no)
+			(do_not_autoplace no)
+			(effects
+				(font
+					(size 1.27 1.27)
+				)
+			)
+		)
+		(property "Value" "+5V"
+			(at 125.73 85.0899 90)
+			(show_name no)
+			(do_not_autoplace no)
+			(effects
+				(font
+					(size 1.27 1.27)
+				)
+				(justify left)
+			)
+		)
+		(property "Footprint" ""
+			(at 129.54 85.09 0)
+			(hide yes)
+			(show_name no)
+			(do_not_autoplace no)
+			(effects
+				(font
+					(size 1.27 1.27)
+				)
+			)
+		)
+		(property "Datasheet" ""
+			(at 129.54 85.09 0)
+			(hide yes)
+			(show_name no)
+			(do_not_autoplace no)
+			(effects
+				(font
+					(size 1.27 1.27)
+				)
+			)
+		)
+		(property "Description" "Power symbol creates a global label with name \"+5V\""
+			(at 129.54 85.09 0)
+			(hide yes)
+			(show_name no)
+			(do_not_autoplace no)
+			(effects
+				(font
+					(size 1.27 1.27)
+				)
+			)
+		)
+		(pin "1"
+		)
+		(instances
+			(project "Kicad Files"
+				(path "/6f8ea6fb-3d53-4ed4-89fa-4890e2ee6e9b"
+					(reference "#PWR035")
+					(unit 1)
+				)
+			)
+		)
+	)
+	(symbol
 		(lib_id "Switch:SW_Push")
 		(at 204.47 96.52 0)
@@
 	)
 	(symbol
-		(lib_id "power:+5V")
-		(at 129.54 82.55 90)
+		(lib_id "power:GND")
+		(at 129.54 82.55 270)
 		(unit 1)
 		(body_style 1)
@@
 		(dnp no)
 		(fields_autoplaced yes)
-		(property "Reference" "#PWR035"
-			(at 133.35 82.55 0)
+		(property "Reference" "#PWR09"
+			(at 123.19 82.55 0)
 			(hide yes)
 			(show_name no)
@@
 			)
 		)
-		(property "Value" "+5V"
+		(property "Value" "GND"
 			(at 125.73 82.5499 90)
 			(show_name no)
@@
 					(size 1.27 1.27)
 				)
-				(justify left)
+				(justify right)
 			)
 		)
@@
 			)
 		)
-		(property "Description" "Power symbol creates a global label with name \"+5V\""
+		(property "Description" "Power symbol creates a global label with name \"GND\" , ground"
 			(at 129.54 82.55 0)
 			(hide yes)
@@
 			(project "Kicad Files"
 				(path "/6f8ea6fb-3d53-4ed4-89fa-4890e2ee6e9b"
-					(reference "#PWR035")
+					(reference "#PWR09")
 					(unit 1)
 				)
@@
 					(unit 1)
 				)
-			)
-		)
-	)
-	(symbol
-		(lib_id "power:GND")
-		(at 129.54 85.09 270)
-		(unit 1)
-		(body_style 1)
-		(exclude_from_sim no)
-		(in_bom yes)
-		(on_board yes)
-		(in_pos_files yes)
-		(dnp no)
-		(fields_autoplaced yes)
-		(property "Reference" "#PWR036"
-			(at 123.19 85.09 0)
-			(hide yes)
-			(show_name no)
-			(do_not_autoplace no)
-			(effects
-				(font
-					(size 1.27 1.27)
-				)
-			)
-		)
-		(property "Value" "GND"
-			(at 125.73 85.0899 90)
-			(show_name no)
-			(do_not_autoplace no)
-			(effects
-				(font
-					(size 1.27 1.27)
-				)
-				(justify right)
-			)
-		)
-		(property "Footprint" ""
-			(at 129.54 85.09 0)
-			(hide yes)
-			(show_name no)
-			(do_not_autoplace no)
-			(effects
-				(font
-					(size 1.27 1.27)
-				)
-			)
-		)
-		(property "Datasheet" ""
-			(at 129.54 85.09 0)
-			(hide yes)
-			(show_name no)
-			(do_not_autoplace no)
-			(effects
-				(font
-					(size 1.27 1.27)
-				)
-			)
-		)
-		(property "Description" "Power symbol creates a global label with name \"GND\" , ground"
-			(at 129.54 85.09 0)
-			(hide yes)
-			(show_name no)
-			(do_not_autoplace no)
-			(effects
-				(font
-					(size 1.27 1.27)
-				)
-			)
-		)
-		(pin "1"
-		)
-		(instances
-			(project "Kicad Files"
-				(path "/6f8ea6fb-3d53-4ed4-89fa-4890e2ee6e9b"
-					(reference "#PWR036")
-					(unit 1)
-				)
